File: audioboard.sch (KiCad schematic (older format))
At the start: 71 parts, among them IC1 TP4054-42-SOT25-R, J1 GCT_USB4085, J2 Conn_01x02, J3 Audio, J4 SJ-43514-SMT, J5 JTAG, J6 UART, J7 GPIO, Q1 AO3401A, SW1 RESET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

Commit message: Add v2
Parts:
- removed C2: 1pF, Capacitor_SMD:C_0402_1005Metric, symbol Device:C
- removed C23: 1uF, Capacitor_SMD:C_0402_1005Metric, symbol Device:C_Small
- removed C30, C31: 47uF, Capacitor_SMD:C_1206_3216Metric, symbol Device:CP_Small
- removed C33, C34: 100nF, Capacitor_SMD:C_0402_1005Metric, symbol Device:C_Small
- removed D3: B5819, Diode_SMD:D_SOD-123, symbol Device:D
- removed J7: GPIO, Connector_PinHeader_2.54mm:PinHeader_1x02_P2.54mm_Vertical, symbol Connector_Generic:Conn_01x02
- removed L2: 4.7nH, Inductor_SMD:L_0402_1005Metric, symbol Device:L
- removed R16: 10k, Resistor_SMD:R_0402_1005Metric, symbol Device:R_Small_US
- added C14: 2.2nF, Capacitor_SMD:C_0402_1005Metric, symbol Device:C_Small
- added C2: 4.7nF, Capacitor_SMD:C_0402_1005Metric, symbol Device:C_Small
- added C3: 10uF, Capacitor_SMD:C_0402_1005Metric, symbol Device:C
- added NT1, NT2: Net-Tie_2, NetTie:NetTie-2_SMD_Pad0.5mm, symbol Device:Net-Tie_2
- added R16: 10k, Resistor_SMD:R_0402_1005Metric, symbol Device:R
- added SW2, SW3: RESET, audioboard:TS1088R02026, symbol Switch:SW_Push
- J1: value GCT_USB4085 -> GCT_USB4125
- J2: footprint Connector_JST:JST_PH_S2B-PH-SM4-TB_1x02-1MP_P2.00mm_Horizontal -> Connector_Molex:Molex_PicoBlade_53261-0271_1x02-1MP_P1.25mm_Horizontal
- J3: footprint Connector_PinHeader_2.54mm:PinHeader_1x06_P2.54mm_Vertical -> Connector_PinHeader_2.54mm:PinHeader_1x03_P2.54mm_Vertical; symbol Connector_Generic:Conn_01x06 -> Connector_Generic:Conn_01x03
- L1: value 2.7nH -> 0nH; LCSC C27123 -> C17168
- R4: footprint Resistor_SMD:R_0603_1608Metric -> Resistor_SMD:R_0402_1005Metric; LCSC C22975 -> C4109
- R5: value 10k -> 3.3k; LCSC C25744 -> C25890
Connections:
- net GPIO19 is gone; now on net STATUS_LED: U2.38 (IO19)
- net LINEOUT_L is gone; now on net LINEIN_L: J3.3 (Pin_3)
- net LINEOUT_R is gone; now on net LINEIN_R: J3.2 (Pin_2)
- net +3V3: now also C3.1, NT2.2; no longer C18.1, C20.1, R6.2, U1.16 (HPVDD), U1.17 (AVDD)
- net ADCVREF: now also C16.1, C7.1; no longer C16.2, C7.2
- net Ant: now also L1.2, C2.2
- net GND: now also C14.1, C2.1, C3.2, NT1.2, SW2.1, SW3.1; no longer C16.1, C17.2, C18.2, C20.2, C7.1, C8.2, J3.1 (Pin_1), J3.4 (Pin_4), J4.4, L1.2, U1.13 (HPGND), U1.18 (AGND)
- net I2S_BCLK: now also U2.16 (IO27); no longer U2.34 (IO5)
- net LINEIN_L: no longer J3.6 (Pin_6)
- net LINEIN_R: no longer J3.5 (Pin_5)
- net STATUS_LED: no longer U2.10 (IO34)
- net VBUS: now also R16.2
- net IO21: now reaches U2.42 (IO21)
- net IO21: now also SW2.2
- net at E1.2, L1.1: now also C14.2
- net at IC1.1 (~CHRG), R4.1: now also R16.1
- net at U1.23 (RIN1): now also C24.2, U1.24 (LIN1)
- net GPIO22 renamed IO22
- net IO22: now also SW3.2
- net VCC: no longer names the net of J5.1 (Pin_1)
- net VCC: no longer J6.2 (Pin_2)
- new net +3.3VA: C18.1, C20.1, NT2.1, R6.2, U1.16 (HPVDD), U1.17 (AVDD)
- new net GNDA: C16.2, C17.2, C18.2, C20.2, C7.2, C8.2, J3.1 (Pin_1), J4.4, NT1.1, U1.13 (HPGND), U1.18 (AGND)
- no-connect marks 19 -> 23
Other:
- moved on the sheet: C10, C12, C13, C15, C16, C17, C18, C20, C4, C5, C6, C7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
